File: final schematic/514final.kicad_sch (KiCad schematic)
At the start: 27 parts, among them M1 Stepper_Motor_unipolar_5pin, M2 Stepper_Motor_unipolar_5pin, U7 MLX90614ESF-BAA-000-TU

Commit message: add second device code
Parts:
- removed C5: 100nF, Capacitor_SMD:C_0603_1608Metric_Pad1.08x0.95mm_HandSolder, symbol Device:C
- removed D1, D2, D4, D5: WS2812B, LED_SMD:LED_WS2812B_PLCC4_5.0x5.0mm_P3.2mm, symbol LED:WS2812B
- removed M1, M2: Stepper_Motor_unipolar_5pin, symbol Motor:Stepper_Motor_unipolar_5pin
- removed OLED1, OLED2: ~, symbol Assignment4:OLED
- removed R14, R9: 3.3kΩ, Resistor_SMD:R_0603_1608Metric_Pad0.98x0.95mm_HandSolder, symbol Device:R
- removed U1: ~, KicadFootprints:XIAO_ESP32, symbol project514:XIAO_ESP32
- removed U2: ~, symbol Assignment4:XIAO_ESP32-C3
- removed U3, U6: ~, symbol project514:rotaryencoder
- removed U7: MLX90614ESF-BAA-000-TU, KicadFootprints:MLX90614ESF-BAA-000-4, symbol project514:MLX90614ESF-BAA-000-TU
- removed piezobuzzer1, piezobuzzer2: ~, symbol Assignment4:piezo_buzzer
- added C1: 100nF, Capacitor_SMD:C_0603_1608Metric_Pad1.08x0.95mm_HandSolder, symbol Device:C
- added R1, R2: 3.3kΩ, Resistor_SMD:R_0603_1608Metric_Pad0.98x0.95mm_HandSolder, symbol Device:R
- added SW1: SW_SPDT, Connector_PinSocket_2.54mm:PinSocket_1x03_P2.54mm_Vertical, symbol Switch:SW_SPDT
- added U2: MLX90614ESF-BAA-000-TU, 514Final:MLX90614ESF-BAA_MEL, symbol 514Final:MLX90614ESF-BAA-000-TU
- BT1: footprint (none) -> Connector_PinSocket_2.54mm:PinSocket_1x02_P2.54mm_Vertical
- U9: footprint KicadFootprints:XIAO_ESP32 -> 514Final:XIAO_ESP32
Connections:
- net +3V3: now also C1.1, R1.2, R2.1, U2.3 (VDD)
- net GND: now also C1.2, U2.4 (VSS)
- net SCL: now also R1.1, U2.1 (SCL/VZ)
- net SDA: now also R2.2, U2.2 (SDA/PWM)
- net at BT1.1 (+): now also SW1.1 (A); no longer U9.15 (+BATT)
- new net: SW1.2 (B), U9.15 (+BATT)
Other:
- note removed: "cooking terminal"
- moved on the sheet: BT1, U9
